File: Schematics/Circuit_Schematicv2.sch (EAGLE design)
At the start: 50 parts, among them Q2 LE33CZ, U1 TDA2822M, U2 23LC1024-I/SN, X1 1502_01

Commit message: Added EEPROM Chip connections, and finished ESP connections
We now need to complete it by adding the DAC and RAM chips if we are
going to use them. Also we should delete the MOSFETs as theyre not
needed anymore
Parts:
- removed DIS1: TUXGR_16X2_R2, display-lcd:TUXGR_16X2_R2
- removed U$2: LCD-HD447804-HOLES20X4-4HOLES, HD44780LCD:LCD-HD447804-HOLES20X4-4HOLES
- added JP2: (no value), MIRO:LCD16X2HEADER
- added R6, R7, R8, R9: 300, SparkFun-Resistors:1OHM-0603-1/10W-1%
- added S3: MOMENTARY-SWITCH-SPST-SMD-6.0X3.5MM, SparkFun-Switches:MOMENTARY-SWITCH-SPST-SMD-6.0X3.5MM
- added VR3: 10k, SparkFun-Resistors:TRIMPOT-SMD-3MM-OPEN-1/10W-25%
Connections:
- removed net N$19: U$2.VO
- removed net N$21: U$2.RS
- removed net N$22: U$2.R/W
- removed net N$23: U$2.E
- new net A: JP2.15, VR3.WIPER
- new net CH_PD: MDL1.CH_PD, R6.1
- new net EN: JP2.6, U$1.RD3/SEG3
- new net K: JP2.16
- new net N$10: R9.2, U$3.WP
- new net REST: MDL1.REST, R7.2, S3.2
- new net RS: JP2.4, U$1.RD2/SEG2
- new net VO: JP2.3
- net 3.3V: now also JP2.2, R6.2, R7.1, U$3.VCC, VR1.CW, VR1.WIPER, VR3.CW; no longer U$2.VDD
- net CLOCK: now also U$3.SCL
- net DATA: now also U$3.SDA
- net DB4: now also JP2.11; no longer U$2.DB4
- net DB5: now also JP2.12; no longer U$2.DB5
- net DB6: now also JP2.13; no longer U$2.DB6
- net DB7: now also JP2.14; no longer U$2.DB7
- net GND: now also JP2.1, JP2.10, JP2.5, JP2.7, JP2.8, JP2.9, MDL1.GPIO15, R8.1, R8.2, R9.1, S3.1, U$3.A0, U$3.A1, U$3.A2, U$3.GND, VR1.CCW, VR3.CCW; no longer U$2.DB0, U$2.DB1, U$2.DB2, U$2.DB3, U$2.VSS
Other:
- note added: "24C64 - EXTERNAL EEPROM CHIP FOR PIC"
- note added: "AR1010 - FM CHIP"
- note added: "ESP8266"
- note added: "HD44780 - 16x2 LCD DISPLAY"
- moved on the sheet: R5, S2, U$3, U$4, U2, UDA1334ATS/N2_ALEX1, VR1

Commit message: added some connectors and cleaned up the code
Parts:
- removed T10, T11, T6, T7, T8, T9: (no value), zetex:NMOSSOT223
- removed U2: 23LC1024-I/SN, microchip_fromOneCall:23LC1024-I/SN
- removed UDA1334ATS/N2_ALEX1: UDA1334ATS/N2_ALEX, UDA1334ATS_ALEX:UDA1334ATS/N2_ALEX
Connections:
- removed net ESPDOWN: MDL1.GPIO4, T9.G
- removed net ESPENABLE: T11.G
- removed net ESPMUTE: MDL1.GPIO9, T10.G
- removed net ESPNEXT: MDL1.GPIO12, T6.G
- removed net ESPPREV: MDL1.GPIO10, T7.G
- removed net ESPUP: MDL1.GPIO5, T8.G
- net ENABLE: no longer T11.D
- net GND: no longer T10.S, T11.S, T6.S, T7.S, T8.S, T9.S
- net MUTE: now also MDL1.GPIO9; no longer T10.D
- net NEXT: now also MDL1.GPIO12; no longer T6.D
- net PREVIOUS: now also MDL1.GPIO10; no longer T7.D
- net VOLDOWN: now also MDL1.GPIO4; no longer T9.D
- net VOLUP: now also MDL1.GPIO5; no longer T8.D
Other:
- note added: "PIC18F6490"
- note removed: "DAC"
- note removed: "RAM"
- moved on the sheet: R9, S10, S11, S12, S7, S8, S9, U$1, U$3

Commit message: added more test pads
Parts:
- removed USB-SERIAL_CONVERTER: (no value), SparkFun-Connectors:CONN_03
- added 3.3V, CLOCK, DATA, GND, L-OUT, TP11: TPSPAD1-13, testpad:TPSPAD1-13
- added AR_PRG: (no value), pinhead:PINHD-1X7
- added ESP_PRG: (no value), pinhead:PINHD-1X3
- added INT_PINS: (no value), pinhead:PINHD-1X2
- added JP3: (no value), pinhead:PINHD-1X8
- added PIC_PRG: (no value), pinhead:PINHD-1X6
- 5V_BAT: value (none) -> 5V
- D1: device SparkFun-LED:LED10MM -> adafruit:LED
Connections:
- removed net N$2: MDL1.TXD, USB-SERIAL_CONVERTER.2
- removed net N$3: MDL1.RXD, USB-SERIAL_CONVERTER.1
- removed net N$7: C7.1, U1.OUT_1
- new net ANT: U$4.ANT
- new net INT2: INT_PINS.1, U$1.RB2/INT2/SEG9
- new net INT3: INT_PINS.2, U$1.RB3/INT3/SEG10
- new net MCLR: PIC_PRG.1, U$1.RG5/~MCLR/VPP
- new net OUT1: C7.1, TP11.PP, U1.OUT_1
- new net PGC: PIC_PRG.5, U$1.RB6/KBI2/PGC
- new net PGD: PIC_PRG.4, U$1.RB7/KBI3/PGD
- new net PGM: PIC_PRG.6
- new net RF0: JP3.1, U$1.RF0/AN5/SEG18
- new net RF1: JP3.2, U$1.RF1/AN6/C2OUT/SEG19
- new net RF2: JP3.3, U$1.RF2/AN7/C1OUT/SEG20
- new net RF3: JP3.4, U$1.RF3/AN8/SEG21
- new net RF4: JP3.5, U$1.RF4/AN9/SEG22
- new net RF5: JP3.6, U$1.RF5/AN10/CVREF/SEG23
- new net RF6: JP3.7, U$1.RF6/AN11/SEG24
- new net RF7: JP3.8, U$1.RF7/~SS/SEG25
- new net RXD: ESP_PRG.2, MDL1.RXD
- new net TXD: ESP_PRG.1, MDL1.TXD
- new net W/R: AR_PRG.5, U$4.W/R
- net 3.3V: now also 3.3V.PP, AR_PRG.1, PIC_PRG.2, U$1.AVDD, U$1.VDD_2, U$1.VDD_3, U$1.VDD_4
- net CLOCK: now also AR_PRG.6, CLOCK.PP
- net DATA: now also AR_PRG.7, DATA.PP
- net ENABLE: now also MDL1.GPIO14
- net GND: now also AR_PRG.2, ESP_PRG.3, GND.PP, PIC_PRG.3, U$1.AVSS, U$1.VSS_2, U$1.VSS_4; no longer USB-SERIAL_CONVERTER.3
- net L-OUT: now also AR_PRG.3, L-OUT.PP
- net N$20: now also 5V_BAT.+@1
- net R-OUT: now also AR_PRG.4
