File: Schematics/Circuit_Schematicv2.sch (EAGLE design)
At the start: 57 parts, among them Q2 LE33CZ, U1 TDA2822M, X1 1502_01

Commit message: started creating PCB
Gonna be tough
Parts:
- removed 5V_BAT: 5V, special:BATTERY
- removed JP3: (no value), pinhead:PINHD-1X8
- removed S1: (no value), switch:255SB
- removed S12: MOMENTARY-SWITCH-SPST-PTH-6.0MM-KIT, SparkFun-Switches:MOMENTARY-SWITCH-SPST-PTH-6.0MM-KIT
- removed U1: TDA2822M, ST Microelctronics_By_element14_Batch_1:TDA2822M
- removed VR2: (no value), SparkFun-Resistors:POTENTIOMETER_DUAL-PTH-12MM-1/20W-20%
- removed X1: 1502_01, con-lumberg:1502_01
- added ANT, BAT_5V, BAT_GND, SWITCH1, SWITCH2: (no value), wirepad:2,15/1,0
- added AUXJACK: (no value), pinhead:PINHD-1X5
- added R10, R16, R17: 10k, SparkFun-Resistors:10KOHM-0603-1/10W-1%
- added S4: FAV1, SparkFun-Switches:MOMENTARY-SWITCH-SPST-PTH-6.0MM-KIT
- added S5: FAV2, SparkFun-Switches:MOMENTARY-SWITCH-SPST-PTH-6.0MM-KIT
- added S6: FAV3, SparkFun-Switches:MOMENTARY-SWITCH-SPST-PTH-6.0MM-KIT
- added SPARE: (no value), pinhead:PINHD-1X8
- added U$2: TDA2822M, smd-footprints:TDA2822M
- added VR4, VR5: 4.7k, SparkFun-Resistors:TRIMPOT-SMD-3MM-OPEN-1/10W-25%
- S10: value MOMENTARY-SWITCH-SPST-PTH-6.0MM-KIT -> VOLDOWN
- S11: value MOMENTARY-SWITCH-SPST-PTH-6.0MM-KIT -> MUTE
- S2: value MOMENTARY-SWITCH-SPST-SMD-6.0X3.5MM -> GPIO0 ESP
- S3: value MOMENTARY-SWITCH-SPST-SMD-6.0X3.5MM -> RESET ESP
- S7: value MOMENTARY-SWITCH-SPST-PTH-6.0MM-KIT -> NEXT
- S8: value MOMENTARY-SWITCH-SPST-PTH-6.0MM-KIT -> PREVIOUS
- S9: value MOMENTARY-SWITCH-SPST-PTH-6.0MM-KIT -> VOLUP
Connections:
- removed net K: JP2.16
- removed net N$1: C5.2, U1.IN-(2)
- removed net N$14: C10.1, C7.2, X1.2
- removed net N$15: C8.1, U1.OUT_2
- removed net N$16: C8.2, C9.1, X1.3
- removed net N$4: U1.IN+(1), VR2G$2.S
- removed net N$5: U1.IN+(2), VR2G$1.S
- removed net N$9: C6.2, U1.IN-(1)
- removed net OUT1: C7.1, TP11.PP, U1.OUT_1
- new net FAV1: MDL1.GPIO16, R10.2, S4.1, U$1.RC5/SDO/SEG12
- new net FAV2: MDL1.GPIO13, R16.2, S5.1, U$1.RC6/TX1/CK1
- new net FAV3: MDL1.GPIO2, R17.2, S6.1, U$1.RC7/RX1/DT1
- new net IN+(1): U$2.IN+(1), VR4.WIPER
- new net IN+(2): U$2.IN+(2), VR5.WIPER
- new net IN-(1): C6.2, U$2.IN-(1)
- new net IN-(2): C5.2, U$2.IN-(2)
- new net N$24: MDL1.GPIO15, R8.2
- new net OUTPUT(1): C7.1, U$2.OUTPUT(1)
- new net OUTPUT(2): C8.1, U$2.OUTPUT(2)
- new net OUT_1: AUXJACK.1, AUXJACK.2, C10.1, C7.2, TP11.PP
- new net OUT_2: AUXJACK.4, AUXJACK.5, C8.2, C9.1
- net 3.3V: now also R10.1, R16.1, R17.1
- net ANT: now also ANT.P
- net ENABLE: no longer S12.1
- net GND: now also AUXJACK.3, BAT_GND.P, JP2.16, S4.2, S5.2, S6.2, U$2.GND, VR4.CCW, VR5.CCW; no longer 5V_BAT.-, MDL1.GPIO15, R8.2, S12.2, U1.GND, VR2G$1.E, VR2G$2.E, X1.1
- net N$11: now also VR5.CW; no longer VR2G$1.A
- net N$12: now also VR4.CW; no longer VR2G$2.A
- net N$20: now also BAT_5V.P, SWITCH2.P; no longer 5V_BAT.+, 5V_BAT.+@1, S1.P
- net RF0: now also SPARE.1; no longer JP3.1
- net RF1: now also SPARE.2; no longer JP3.2
- net RF2: now also SPARE.3; no longer JP3.3
- net RF3: now also SPARE.4; no longer JP3.4
- net RF4: now also SPARE.5; no longer JP3.5
- net RF5: now also SPARE.6; no longer JP3.6
- net RF6: now also SPARE.7; no longer JP3.7
- net RF7: now also SPARE.8; no longer JP3.8
- net VDD: now also SWITCH1.P, U$2.VDD; no longer S1.O, U1.SUPPLY_VOLTAGE
Other:
- note added: "SPARE PINS AND TEST POINTS"

Commit message: very close to finishing the PCB design. Very tiny!
Connections:
- new net N$51: JP2.2, VR1.WIPER
- net 3.3V: no longer JP2.2, VR1.WIPER
Changed lines of the file:
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@@
-</segment>
-<segment>
-<pinref part="JP2" gate="A" pin="2"/>
-<label x="17.78" y="-43.18" size="1.778" layer="95" rot="R180"/>
-<pinref part="VR1" gate="R?" pin="WIPER"/>
-<wire x1="7.62" y1="-43.18" x2="33.02" y2="-43.18" width="0.1524" layer="91"/>
-<wire x1="33.02" y1="-43.18" x2="33.02" y2="-45.72" width="0.1524" layer="91"/>
 </segment>
 <segment>
@@
 </segment>
 </net>
+<net name="N$51" class="0">
+<segment>
+<pinref part="JP2" gate="A" pin="2"/>
+<label x="17.78" y="-43.18" size="1.778" layer="95" rot="R180"/>
+<pinref part="VR1" gate="R?" pin="WIPER"/>
+<wire x1="7.62" y1="-43.18" x2="33.02" y2="-43.18" width="0.1524" layer="91"/>
+<wire x1="33.02" y1="-43.18" x2="33.02" y2="-45.72" width="0.1524" layer="91"/>
+</segment>
+</net>

Commit message: recent eagle changes
Connections:
- new net N$1: U$1.AVDD, U$1.VDD
- net 3.3V: no longer U$1.AVDD, U$1.VDD, U$1.VDD_3, U$1.VDD_4
- net GND: no longer U$1.VSS_2, U$1.VSS_3, U$1.VSS_4
