File: Schematics/Circuit_Schematicv2.brd (EAGLE design)
At the start: 139.1 x 33.1 mm, 66 parts, among them Q2 LE33CZ

Commit message: very close to finishing the PCB design. Very tiny!
Parts:
- moved PIC_PRG 53.3 mm to (-6.60, 20.8), turned to 0 degrees
- moved C3 49.9 mm to (12.1, 28.4), turned to 90 degrees
- moved TP11 39.8 mm to (-54.4, 49.1)
- moved ESP_PRG 39.6 mm to (50.7, 20.7), turned to 180 degrees
- moved U$1 29.7 mm to (-13.8, 35.9)
- moved U$4 29.4 mm to (13.7, 35.8), turned to 180 degrees
- moved INT_PINS 28.3 mm to (-4.57, 48.5)
- moved R5 20.6 mm to (45.3, 24.9)
- moved ANT 20.5 mm to (5.08, 27.4)
- moved R7 16.0 mm to (31.4, 24.9)
- moved R6 15.8 mm to (38.1, 25.0), turned to 0 degrees
- moved C9 14.7 mm to (-69.5, 35.3), flipped to the bottom, turned to 180 degrees
- moved R2 14.3 mm to (-25.9, 40.5), turned to 180 degrees
- moved C10 13.7 mm to (-54.7, 36.8), flipped to the bottom, turned to 270 degrees
- moved VR1 9.94 mm to (-39.9, 21.2)
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Connections:
- new net N$51: JP2.2, VR1.2
- net 3.3V: no longer JP2.2, VR1.2
Routing:
- net GND: track 15.9 -> 367.6 mm, vias 0 -> 4
- net 3.3V: track 0.00 -> 247.3 mm, vias 0 -> 10
- net FAV2: track 0.00 -> 138.4 mm, vias 0 -> 3
- net FAV1: track 0.00 -> 122.7 mm, vias 0 -> 7
- net FAV3: track 0.00 -> 118.7 mm, vias 0 -> 11
- net PREVIOUS: track 0.00 -> 105.7 mm, vias 0 -> 9
- net N$51: track 0.00 -> 105.4 mm, vias 0 -> 8
- net MUTE: track 0.00 -> 103.0 mm, vias 0 -> 4
- net VOLUP: track 0.00 -> 99.9 mm, vias 0 -> 8
- net VOLDOWN: track 0.00 -> 95.6 mm, vias 0 -> 5
- net L-OUT: track 0.00 -> 85.9 mm, vias 0 -> 5
- net DATA: track 0.00 -> 79.1 mm, vias 0 -> 5
- net A: track 0.00 -> 78.6 mm, vias 0 -> 6
- net NEXT: track 0.00 -> 76.1 mm, vias 0 -> 4
- net CLOCK: track 0.00 -> 73.8 mm, vias 0 -> 5
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Other:
- outline, holes or cut-outs redrawn

Commit message: recent eagle changes
Parts:
- moved DATA 5.72 mm to (-3.17, 49.0)
- moved INT_PINS 3.83 mm to (-8.38, 48.9)
- moved CLOCK 1.14 mm to (-12.4, 48.9)
Connections:
- new net N$1: U$1.19, U$1.57
- new net VDD_3: U$1.38
- new net VDD_4: U$1.10
- new net VSS_2: U$1.41
- new net VSS_3: U$1.56
- new net VSS_4: U$1.25
- net 3.3V: no longer U$1.10, U$1.19, U$1.38, U$1.57
- net GND: no longer U$1.25, U$1.41, U$1.56
Routing:
- net DATA: track 79.1 -> 73.4 mm
- net GND: track 367.6 -> 364.0 mm
- net L-OUT: track 85.9 -> 84.1 mm
- net CLOCK: track 73.8 -> 73.3 mm
Changed lines of the file:
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@@
 <attribute name="PROD_ID" value="CAP-09824" x="-69.469" y="35.306" size="1.778" layer="28" rot="MR180" display="off"/>
 </element>
-<element name="CLOCK" library="testpad" package="P1-13" value="TPSPAD1-13" x="-11.303" y="48.895">
-<attribute name="TP_SIGNAL_NAME" value="" x="-11.303" y="48.895" size="1.778" layer="27" display="off"/>
+<element name="CLOCK" library="testpad" package="P1-13" value="TPSPAD1-13" x="-12.446" y="48.895">
+<attribute name="TP_SIGNAL_NAME" value="" x="-12.446" y="48.895" size="1.778" layer="27" display="off"/>
 </element>
 <element name="D1" library="adafruit" package="SMARTLED-TTW" value="" x="-78.994" y="20.701" rot="R270"/>
-<element name="DATA" library="testpad" package="P1-13" value="TPSPAD1-13" x="-8.89" y="48.895">
-<attribute name="TP_SIGNAL_NAME" value="" x="-8.89" y="48.895" size="1.778" layer="27" display="off"/>
+<element name="DATA" library="testpad" package="P1-13" value="TPSPAD1-13" x="-3.175" y="49.022">
+<attribute name="TP_SIGNAL_NAME" value="" x="-3.175" y="49.022" size="1.778" layer="27" display="off"/>
 </element>
 <element name="ESP_PRG" library="pinhead" package="1X03" value="" x="50.673" y="20.701" rot="R180"/>
@@
 <attribute name="TP_SIGNAL_NAME" value="" x="-18.034" y="48.895" size="1.778" layer="27" display="off"/>
 </element>
-<element name="INT_PINS" library="pinhead" package="1X02" value="" x="-4.572" y="48.514"/>
+<element name="INT_PINS" library="pinhead" package="1X02" value="" x="-8.382" y="48.895"/>
 <element name="JP2" library="MIRO" package="LCD16X2HEADER" value="" x="27.94" y="47.625" rot="MR0"/>
 <element name="L-OUT" library="testpad" package="P1-13" value="TPSPAD1-13" x="-15.494" y="48.895">
@@
 <contactref element="R1" pad="1"/>
 <contactref element="U$1" pad="9"/>
-<contactref element="U$1" pad="56"/>
-<contactref element="U$1" pad="41"/>
 <contactref element="U$1" pad="20"/>
-<contactref element="U$1" pad="25"/>
 <contactref element="S7" pad="3"/>
 <contactref element="S8" pad="3"/>
@@
 <wire x1="-0.3175" y1="36.98875" x2="-0.381" y2="37.0332" width="0.254" layer="1"/>
 <wire x1="-3.81" y1="36.195" x2="-4.445" y2="36.195" width="0.254" layer="1"/>
-<wire x1="-4.445" y1="36.195" x2="-8.1026" y2="36.195" width="0.254" layer="1"/>
 <wire x1="-3.01625" y1="36.98875" x2="-3.81" y2="36.195" width="0.254" layer="1"/>
 <wire x1="-3.01625" y1="36.98875" x2="-2.921" y2="37.0332" width="0.254" layer="1"/>
@@
 <via x="-8.5725" y="29.5275" extent="1-16" drill="0.6096"/>
 <via x="-17.145" y="34.76625" extent="1-16" drill="0.6096"/>
-<wire x1="-8.1026" y1="36.195" x2="-13.589" y2="41.6814" width="0" layer="19" extent="1-1"/>
-<wire x1="-13.589" y1="30.2006" x2="-11.27125" y2="29.5275" width="0" layer="19" extent="1-16"/>
-<wire x1="-16.1036" y1="30.2006" x2="-13.589" y2="30.2006" width="0" layer="19" extent="1-1"/>
+<wire x1="-15.08125" y1="32.54375" x2="-16.1036" y2="30.2006" width="0" layer="19" extent="1-16"/>
 </signal>
 <signal name="N$11">
@@
 <wire x1="16.66875" y1="34.44875" x2="12.54125" y2="34.44875" width="0.254" layer="1"/>
 <wire x1="16.66875" y1="34.44875" x2="16.716" y2="34.314" width="0.254" layer="1"/>
-<wire x1="-8.5725" y1="48.895" x2="-8.89" y2="48.895" width="0.254" layer="16"/>
-<wire x1="-6.19125" y1="46.51375" x2="-8.5725" y2="48.895" width="0.254" layer="16"/>
-<wire x1="-1.5875" y1="46.51375" x2="-6.19125" y2="46.51375" width="0.254" layer="16"/>
-<wire x1="0" y1="48.10125" x2="-1.5875" y2="46.51375" width="0.254" layer="16"/>
-<wire x1="3.33375" y1="48.10125" x2="0" y2="48.10125" width="0.254" layer="16"/>
 <wire x1="8.09625" y1="43.33875" x2="3.33375" y2="48.10125" width="0.254" layer="1"/>
 <wire x1="8.09625" y1="42.06875" x2="8.09625" y2="43.33875" width="0.254" layer="1"/>
@@
 <via x="12.54125" y="34.44875" extent="1-16" drill="0.6096"/>
 <via x="3.33375" y="48.10125" extent="1-16" drill="0.6096"/>
+<wire x1="-2.25425" y1="48.10125" x2="-3.175" y2="49.022" width="0.254" layer="16"/>
+<wire x1="-3.175" y1="49.022" x2="-2.25425" y2="48.10125" width="0.254" layer="16"/>
+<wire x1="-2.25425" y1="48.10125" x2="3.33375" y2="48.10125" width="0.254" layer="16"/>
 </signal>
 <signal name="CLOCK">
@@
 <wire x1="18.57375" y1="20.79625" x2="18.542" y2="20.701" width="0.254" layer="16"/>
 <wire x1="-9.68375" y1="32.7025" x2="-8.255" y2="32.7025" width="0.254" layer="1"/>
-<wire x1="-6.985" y1="32.7025" x2="-7.62" y2="32.7025" width="0.254" layer="16"/>
+<wire x1="-7.62" y1="32.7025" x2="-6.985" y2="32.7025" width="0.254" layer="16"/>
 <wire x1="-7.62" y1="32.7025" x2="-9.68375" y2="32.7025" width="0.254" layer="16"/>
-<wire x1="-5.55625" y1="31.27375" x2="-6.985" y2="32.7025" width="0.254" layer="16"/>
+<wire x1="-6.985" y1="32.7025" x2="-5.55625" y2="31.27375" width="0.254" layer="16"/>
 <wire x1="-4.1275" y1="31.27375" x2="-5.55625" y2="31.27375" width="0.254" layer="16"/>
 <wire x1="-1.74625" y1="33.655" x2="-3.730625" y2="31.670625" width="0.254" layer="16"/>
@@
 <wire x1="-8.255" y1="32.7025" x2="-8.1026" y2="32.6898" width="0.254" layer="1"/>
 <wire x1="-1.74625" y1="31.90875" x2="-1.651" y2="31.8008" width="0.254" layer="1"/>
-<wire x1="-11.43" y1="45.72" x2="-11.43" y2="48.895" width="0.254" layer="1"/>
-<wire x1="-12.54125" y1="44.60875" x2="-11.43" y2="45.72" width="0.254" layer="1"/>
-<wire x1="-12.54125" y1="43.18" x2="-12.54125" y2="44.60875" width="0.254" layer="1"/>
-<wire x1="-12.54125" y1="37.62375" x2="-12.54125" y2="43.18" width="0.254" layer="16"/>
-<wire x1="-7.62" y1="32.7025" x2="-12.54125" y2="37.62375" width="0.254" layer="16"/>
-<wire x1="-11.43" y1="48.895" x2="-11.303" y2="48.895" width="0.254" layer="1"/>
+<wire x1="-12.54125" y1="43.18" x2="-12.54125" y2="37.62375" width="0.254" layer="16"/>
 <wire x1="14.76375" y1="36.195" x2="16.66875" y2="36.195" width="0.254" layer="1"/>
 <wire x1="13.97" y1="35.40125" x2="14.76375" y2="36.195" width="0.254" layer="1"/>
@@
 <via x="-12.54125" y="43.18" extent="1-16" drill="0.6096"/>
 <via x="13.97" y="35.40125" extent="1-16" drill="0.6096"/>
+<wire x1="-12.54125" y1="43.18" x2="-12.446" y2="43.27525" width="0.254" layer="1"/>
+<wire x1="-12.446" y1="43.27525" x2="-12.446" y2="48.895" width="0.254" layer="1"/>
+<wire x1="-7.62" y1="32.7025" x2="-12.54125" y2="37.62375" width="0.254" layer="16"/>
 </signal>
 <signal name="IN+(1)">
@@
 <contactref element="MDL1" pad="8"/>
 <contactref element="U$4" pad="VCC"/>
-<contactref element="U$1" pad="57"/>
-<contactref element="U$1" pad="19"/>
 <contactref element="U$1" pad="26"/>
-<contactref element="U$1" pad="10"/>
-<contactref element="U$1" pad="38"/>
 <contactref element="R5" pad="1"/>
 <contactref element="VR1" pad="1"/>
@@
 <wire x1="-18.494375" y1="47.069375" x2="-14.12875" y2="42.70375" width="0.254" layer="1"/>
 <wire x1="-20.574" y1="48.895" x2="-20.32" y2="48.895" width="0.254" layer="1"/>
-<wire x1="-14.12875" y1="41.75125" x2="-14.097" y2="41.6814" width="0.254" layer="1"/>
 <wire x1="-26.67" y1="33.655" x2="-26.67" y2="32.54375" width="0.254" layer="16"/>
 <wire x1="-25.0825" y1="35.2425" x2="-26.67" y2="33.655" width="0.254" layer="16"/>
@@
 <via x="-5.23875" y="23.65375" extent="1-16" drill="0.6096"/>
 <via x="-6.985" y="22.86" extent="1-16" drill="0.6096"/>
-<wire x1="-13.081" y1="30.2006" x2="-8.1026" y2="34.6964" width="0" layer="19" extent="1-1"/>
-<wire x1="-16.5862" y1="30.2006" x2="-13.081" y2="30.2006" width="0" layer="19" extent="1-1"/>
-<wire x1="-19.20875" y1="30.1625" x2="-16.5862" y2="30.2006" width="0" layer="19" extent="1-16"/>
-<wire x1="-19.5834" y1="35.179" x2="-19.20875" y2="30.1625" width="0" layer="19" extent="1-16"/>
+<wire x1="-13.97" y1="24.92375" x2="-13.081" y2="30.2006" width="0" layer="19" extent="1-16"/>
 </signal>
 <signal name="L-OUT">
@@
 <wire x1="-11.90625" y1="36.195" x2="-17.145" y2="41.43375" width="0.254" layer="16"/>
 <wire x1="-11.90625" y1="33.81375" x2="-11.90625" y2="36.195" width="0.254" layer="16"/>
-<wire x1="-10.63625" y1="32.54375" x2="-11.90625" y2="33.81375" width="0.254" layer="1"/>
+<wire x1="-10.63625" y1="32.54375" x2="-11.90625" y2="33.81375" width="0" layer="19" extent="1-16"/>
 <wire x1="-10.63625" y1="32.385" x2="-10.63625" y2="32.54375" width="0.254" layer="1"/>
 <wire x1="-9.8425" y1="31.59125" x2="-10.63625" y2="32.385" width="0.254" layer="1"/>
@@
 <contactref element="U$1" pad="46"/>
 <contactref element="INT_PINS" pad="1"/>
-<wire x1="-8.1026" y1="38.6842" x2="-5.842" y2="48.514" width="0" layer="19" extent="1-1"/>
+<wire x1="-8.1026" y1="38.6842" x2="-9.652" y2="48.895" width="0" layer="19" extent="1-1"/>
 </signal>
 <signal name="INT3">
 <contactref element="U$1" pad="45"/>
 <contactref element="INT_PINS" pad="2"/>
-<wire x1="-8.1026" y1="38.2016" x2="-3.302" y2="48.514" width="0" layer="19" extent="1-1"/>
+<wire x1="-8.1026" y1="38.2016" x2="-7.112" y2="48.895" width="0" layer="19" extent="1-1"/>
 </signal>
 <signal name="W/R">
@@
 <via x="15.5575" y="45.72" extent="1-16" drill="0.6096"/>
 </signal>
+<signal name="VSS_4">
+<contactref element="U$1" pad="25"/>
+</signal>
+<signal name="VSS_3">
+<contactref element="U$1" pad="56"/>
+</signal>
+<signal name="VSS_2">
+<contactref element="U$1" pad="41"/>
+</signal>
+<signal name="N$1">
+<contactref element="U$1" pad="57"/>
+<contactref element="U$1" pad="19"/>
+<wire x1="-16.5862" y1="30.2006" x2="-14.097" y2="41.6814" width="0" layer="19" extent="1-1"/>
+</signal>
+<signal name="VDD_4">
+<contactref element="U$1" pad="10"/>
+</signal>
+<signal name="VDD_3">
+<contactref element="U$1" pad="38"/>
+</signal>
 </signals>
