File: Schematics/Circuit_Schematicv2.brd (EAGLE design)
At the start: 139.1 x 33.1 mm, 73 parts, among them Q2 LE33CZ

Commit message: Added GPIO jumpers instead of switches
Parts:
- removed S2: GPIO0 ESP, SparkFun-Switches:TACTILE_SWITCH_SMD_6.0X3.5MM
- added JP1, JP3: (no value), jumper:JP1
Connections:
- new net ESP_VCC: JP1.1, MDL1.8
- net 3.3V: now also JP1.2; no longer MDL1.8
- net ESP_GPIO0: now also JP3.1; no longer S2.2
- net GND: now also JP3.2; no longer S2.1
Routing:
- net 3.3V: track 292.3 -> 284.6 mm
Changed lines of the file:
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@@
 <?xml version="1.0" encoding="utf-8"?>
 <!DOCTYPE eagle SYSTEM "eagle.dtd">
-<eagle version="8.1.0">
+<eagle version="8.0.0">
 <drawing>
 <settings>
@@
 <attribute name="SF_SKU" value="COM-00097 " x="-62.23" y="26.67" size="1.778" layer="28" rot="MR0" display="off"/>
 </element>
-<element name="S2" library="SparkFun-Switches" package="TACTILE_SWITCH_SMD_6.0X3.5MM" value="GPIO0 ESP" x="52.197" y="31.623" rot="R270">
-<attribute name="PROD_ID" value="SWCH-00815" x="52.197" y="31.623" size="1.778" layer="27" rot="R270" display="off"/>
-<attribute name="SF_SKU" value="COM-08229" x="52.197" y="31.623" size="1.778" layer="27" rot="R270" display="off"/>
-</element>
 <element name="S3" library="SparkFun-Switches" package="TACTILE_SWITCH_SMD_6.0X3.5MM" value="RESET ESP" x="52.197" y="41.021" rot="R90">
 <attribute name="PROD_ID" value="SWCH-00815" x="52.197" y="41.021" size="1.778" layer="27" rot="R90" display="off"/>
@@
 <attribute name="OC_NEWARK" value="unknown" x="-85.8266" y="-64.135" size="1.778" layer="27" display="off"/>
 </element>
+<element name="JP1" library="jumper" package="JP1" value="" x="-98.9584" y="-62.5602"/>
+<element name="JP3" library="jumper" package="JP1" value="" x="-113.1824" y="-62.5602"/>
 </elements>
 <signals>
@@
 <contactref element="MDL1" pad="9"/>
 <contactref element="S11" pad="3"/>
-<contactref element="S2" pad="1"/>
 <contactref element="JP2" pad="1"/>
 <contactref element="JP2" pad="5"/>
@@
 <wire x1="26.67" y1="47.625" x2="24.13" y2="47.625" width="0.2032" layer="1"/>
 <wire x1="52.22875" y1="37.7825" x2="52.22875" y2="34.925" width="0.2032" layer="1"/>
-<wire x1="52.22875" y1="34.925" x2="52.197" y2="34.773" width="0.2032" layer="1"/>
 <wire x1="52.22875" y1="37.7825" x2="52.197" y2="37.871" width="0.2032" layer="1"/>
 <wire x1="31.75" y1="47.625" x2="29.21" y2="47.625" width="0.2032" layer="1"/>
@@
 <wire x1="52.22875" y1="34.76625" x2="53.34" y2="33.655" width="0.2032" layer="1"/>
 <wire x1="52.22875" y1="24.92375" x2="52.158" y2="24.892" width="0.2032" layer="1"/>
-<wire x1="52.22875" y1="34.76625" x2="52.197" y2="34.773" width="0.2032" layer="1"/>
 <wire x1="10.795" y1="49.53" x2="8.89" y2="47.625" width="0.2032" layer="16"/>
 <wire x1="22.225" y1="49.53" x2="10.795" y2="49.53" width="0.2032" layer="16"/>
@@
 <contactref element="T6" pad="3"/>
 <contactref element="T7" pad="3"/>
-<wire x1="-83.5152" y1="-56.1086" x2="-83.5152" y2="-67.2338" width="0" layer="19" extent="1-1"/>
+<contactref element="JP3" pad="2"/>
+<wire x1="-83.5152" y1="-56.1086" x2="-113.1824" y2="-61.2902" width="0" layer="19" extent="1-1"/>
+<wire x1="-83.5152" y1="-67.2338" x2="-83.5152" y2="-56.1086" width="0" layer="19" extent="1-1"/>
 <wire x1="-83.5152" y1="-44.9834" x2="-83.5152" y2="-56.1086" width="0" layer="19" extent="1-1"/>
 <wire x1="-83.5152" y1="-33.8582" x2="-83.5152" y2="-44.9834" width="0" layer="19" extent="1-1"/>
@@
 <wire x1="-83.5152" y1="-0.4826" x2="-83.5152" y2="-11.6078" width="0" layer="19" extent="1-1"/>
 <wire x1="-72.5932" y1="21.6526" x2="-83.5152" y2="-0.4826" width="0" layer="19" extent="1-1"/>
+<wire x1="52.22875" y1="34.925" x2="52.22875" y2="34.76625" width="0" layer="19" extent="1-1"/>
 </signal>
 <signal name="N$11">
@@
 <signal name="3.3V">
 <contactref element="Q2" pad="1"/>
-<contactref element="MDL1" pad="8"/>
 <contactref element="U$4" pad="VCC"/>
 <contactref element="U$1" pad="26"/>
@@
 <wire x1="-20.6375" y1="48.895" x2="-20.574" y2="48.895" width="0.2032" layer="1"/>
 <wire x1="-25.4" y1="40.9575" x2="-25.058" y2="40.513" width="0.2032" layer="16"/>
-<wire x1="19.05" y1="44.45" x2="26.765" y2="44.45" width="0.2032" layer="1"/>
 <wire x1="16.8275" y1="42.2275" x2="19.05" y2="44.45" width="0.2032" layer="1"/>
 <wire x1="16.8275" y1="42.2275" x2="16.716" y2="42.314" width="0.2032" layer="1"/>
@@
 <wire x1="-14.986" y1="36.195" x2="-14.986" y2="33.5026" width="0.2032" layer="1"/>
 <wire x1="-14.986" y1="33.5026" x2="-16.5862" y2="31.9024" width="0.2032" layer="1"/>
-<wire x1="-13.081" y1="30.2006" x2="-16.5862" y2="30.2006" width="0" layer="19" extent="1-1"/>
+<contactref element="JP1" pad="2"/>
+<wire x1="-56.67375" y1="20.47875" x2="-98.9584" y2="-61.2902" width="0" layer="19" extent="16-16"/>
+<wire x1="-16.5862" y1="30.2006" x2="-13.081" y2="30.2006" width="0" layer="19" extent="1-1"/>
 </signal>
 <signal name="L-OUT">
@@
 <contactref element="MDL1" pad="12"/>
 <contactref element="R5" pad="2"/>
-<contactref element="S2" pad="2"/>
 <wire x1="48.26" y1="24.92375" x2="46.19625" y2="24.92375" width="0.2032" layer="1"/>
 <wire x1="51.7525" y1="28.41625" x2="48.26" y2="24.92375" width="0.2032" layer="1"/>
 <wire x1="52.07" y1="28.41625" x2="51.7525" y2="28.41625" width="0.2032" layer="1"/>
 <wire x1="46.19625" y1="24.92375" x2="46.189" y2="24.892" width="0.2032" layer="1"/>
-<wire x1="52.07" y1="28.41625" x2="52.197" y2="28.473" width="0.2032" layer="1"/>
 <wire x1="32.86125" y1="26.51125" x2="32.86125" y2="28.09875" width="0.2032" layer="1"/>
 <wire x1="44.45" y1="26.51125" x2="32.86125" y2="26.51125" width="0.2032" layer="16"/>
@@
 <via x="32.86125" y="26.51125" extent="1-16" drill="0.6096"/>
 <via x="44.45" y="26.51125" extent="1-16" drill="0.6096"/>
+<contactref element="JP3" pad="1"/>
+<wire x1="32.86125" y1="26.51125" x2="-113.1824" y2="-63.8302" width="0" layer="19" extent="1-1"/>
+</signal>
+<signal name="ESP_VCC">
+<contactref element="MDL1" pad="8"/>
+<contactref element="JP1" pad="1"/>
+<wire x1="26.765" y1="44.45" x2="-98.9584" y2="-63.8302" width="0" layer="19" extent="1-1"/>
 </signal>
 </signals>
